File: LATE Destilador Shield.sch (KiCad schematic (older format))
At the start: 38 parts, among them J1 PWRSRC, J2 MOTOR_A, J3 MOTOR_B, J4 AC_BUS, J5 LOAD, J6 MOTOR_PWR, Q1 BT136-500, U1 AD620, U2 L298P, U3 MOC3020M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

Commit message: Project upgrade to KiCAD 5.02
Parts:
- J1: symbol conn:Conn_02x02_Top_Bottom -> LATE-Destilador-Shield-rescue:Conn_02x02_Top_Bottom-conn
- J2, J3, J4, J5, J6: symbol conn:Conn_01x02 -> LATE-Destilador-Shield-rescue:Conn_01x02-conn
- U1: symbol linear:AD620 -> LATE-Destilador-Shield-rescue:AD620-linear
- U2: symbol motor_drivers:L298P -> LATE-Destilador-Shield-rescue:L298P-motor_drivers
- U3: symbol opto:MOC3020M -> LATE-Destilador-Shield-rescue:MOC3020M-opto
- U4: symbol opto:4N25 -> LATE-Destilador-Shield-rescue:4N25-opto
Changed lines of the file:
@@
 Shield para Arduino Mega (Destilador LATE)
 $Comp
-L motor_drivers:L298P U2
+L LATE-Destilador-Shield-rescue:L298P-motor_drivers U2
 U 1 1 5A56CAC5
 P 8000 2300
@@
 $EndComp
 $Comp
-L linear:AD620 U1
+L LATE-Destilador-Shield-rescue:AD620-linear U1
 U 1 1 5A5A9575
 P 3300 2800
@@
 $EndComp
 $Comp
-L conn:Conn_02x02_Top_Bottom J1
+L LATE-Destilador-Shield-rescue:Conn_02x02_Top_Bottom-conn J1
 U 1 1 5A5A9E34
 P 2550 1350
@@
 5VDC
 $Comp
-L conn:Conn_01x02 J2
+L LATE-Destilador-Shield-rescue:Conn_01x02-conn J2
 U 1 1 5A5AA409
 P 9950 2100
@@
 $EndComp
 $Comp
-L conn:Conn_01x02 J3
+L LATE-Destilador-Shield-rescue:Conn_01x02-conn J3
 U 1 1 5A5AA462
 P 10250 2400
@@
 $EndComp
 $Comp
-L opto:4N25 U4
+L LATE-Destilador-Shield-rescue:4N25-opto U4
 U 1 1 5A5BA1BB
 P 3200 4700
@@
 $EndComp
 $Comp
-L conn:Conn_01x02 J4
+L LATE-Destilador-Shield-rescue:Conn_01x02-conn J4
 U 1 1 5A5BA8A1
 P 1050 4650
@@
 $EndComp
 $Comp
-L opto:MOC3020M U3
+L LATE-Destilador-Shield-rescue:MOC3020M-opto U3
 U 1 1 5A5BBB3D
 P 2350 6250
@@
 AC1
 $Comp
-L conn:Conn_01x02 J5
+L LATE-Destilador-Shield-rescue:Conn_01x02-conn J5
 U 1 1 5A5BCE5C
 P 4100 6350
@@
 $EndComp
 $Comp
-L conn:Conn_01x02 J6
+L LATE-Destilador-Shield-rescue:Conn_01x02-conn J6
 U 1 1 5A5BAE99
 P 8300 4400
